Commit message: lepiej niż było

File: zad2/urdf/joints_blocked.urdf (robot description, URDF)
Before this commit: robot manipulator, 4 links, 3 joints
Links:
- added link hand; visual cylinder length=0.05 radius=0.02
- link base_link: geometry visual cylinder length=0.1 radius=0.3
Joints:
- added joint link3_to_hand: type fixed, parent link_3, child hand, origin xyz=0 0 0 rpy=0 0 0

File: zad2/urdf/joints_movable.urdf (robot description, URDF)
Before this commit: robot manipulator, 4 links, 3 joints
Links:
- added link hand; visual cylinder length=0.05 radius=0.02
- link base_link: geometry visual cylinder length=0.1 radius=0.3
Joints:
- added joint link3_to_hand: type fixed, parent link_3, child hand, origin xyz=0 0 0 rpy=0 0 0

Commit message: zmiany estetyczne

File: zad2/urdf/joints_blocked.urdf (robot description, URDF)
Before this commit: robot manipulator, 5 links, 4 joints
Links:
- link hand: geometry visual cylinder length=0.05 radius=0.1

File: zad2/urdf/joints_movable.urdf (robot description, URDF)
Before this commit: robot manipulator, 5 links, 4 joints
Links:
- link hand: geometry visual cylinder length=0.05 radius=0.1
